Commit message: add macro for leg. 4 joints done

File: src/mit_cheetah_gazebo/description/test_mini.urdf (robot description, URDF)
Before this commit: robot test_mini, 2 links, 1 joints
Links:
- removed link link_lower
- added link link_root
Joints:
- removed joint one
- added joint root_to_body: type fixed, parent link_root, child link_body, origin xyz=0 0 0 rpy=0 0 0
